File: 328RFStamp.sch (KiCad schematic (older format))
At the start: 20 parts, among them IC1 CC1101, J1 5, J10 RST, J11 14, J13 15, J2 7, J3 8, J4 9, J5 4, J6 6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

Commit message: corrected value for C3
Parts:
- C3: value 22µ -> 10µ
Changed lines of the file:
@@
 P 4920 1890
 F 0 "C3" V 4665 1890 50  0000 C CNN
-F 1 "22µ" V 4756 1890 50  0000 C CNN
+F 1 "10µ" V 4756 1890 50  0000 C CNN
 F 2 "Capacitor_Tantalum_SMD:CP_EIA-3216-18_Kemet-A_Pad1.58x1.35mm_HandSolder" H 4958 1740 50  0001 C CNN
 F 3 "~" H 4920 1890 50  0001 C CNN
