File: 328RFStamp.kicad_pcb (KiCad board)
At the start: 2 copper layers, 17 x 19 mm, 20 parts, among them IC1 CC1101, J1 5, J10 RST, J11 14, J13 15, J2 7, J3 8, J4 9, J5 4, J6 6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

Commit message: update to KiCad 6
Other:
- net class Default removed
